Commit message: Update clover4.xacro

File: clover_description/urdf/clover/clover4.xacro (robot description, xacro)
@@ -1,14 +1,22 @@
 <?xml version="1.0"?>
-<robot name="clover" xmlns:xacro="http://ros.org/wiki/xacro">
+<robot name="clover_camera" xmlns:xacro="http://ros.org/wiki/xacro">
   <xacro:arg name="main_camera" default="true"/>
   <xacro:arg name="rangefinder" default="true"/>
   <xacro:arg name="led" default="true"/>
   <xacro:arg name="gps" default="true"/>
+  <xacro:arg name="d435" default="true"/>
   <xacro:arg name="maintain_camera_rate" default="false"/>
   <xacro:arg name="use_clover_physics" default="false"/>
-  <xacro:include filename="clover4_base.xacro" />
-  <xacro:include filename="../sensors/rpi_cam.urdf.xacro"/>
-  <xacro:include filename="../sensors/distance_sensor.urdf.xacro"/>
-  <xacro:include filename="../leds/led_strip.xacro"/>
+  <xacro:include filename="$(find clover_description)/urdf/clover/clover4_base.xacro" />
+  <xacro:include filename="$(find clover_description)/urdf/sensors/rpi_cam.urdf.xacro"/>
+  <xacro:include filename="$(find clover_description)/urdf/sensors/distance_sensor.urdf.xacro"/>
+  <xacro:include filename="$(find clover_description)/urdf/leds/led_strip.xacro"/>
+  <!-- Use Intel Realsense D455 -->
+  <xacro:include filename="$(find realsense2_description_px4)/urdf/_d435.urdf.xacro"/>
+  <xacro:if value="$(arg d455)">
+    <xacro:sensor_d435 name="camera" topics_ns="camera" parent="base_link" publish_pointcloud="true">
+      <origin xyz="0 0 0.2" rpy="0 0 0" />
+    </xacro:sensor_d435>
+  </xacro:if>
   <!-- Create camera plugin -->
   <xacro:if value="$(arg main_camera)">
@@ -31,15 +39,9 @@
   </xacro:if>
   <xacro:if value="$(arg gps)">
-    <gazebo>
-      <include>
-        <uri>model://gps</uri>
-        <pose>0.1 0 0 0 0 0</pose>
-        <name>gps0</name>
-      </include>
-      <joint name='gps0_joint' type='fixed'>
-        <child>gps0::link</child>
-        <parent>base_link</parent>
-      </joint>
-    </gazebo>
+    <!-- Instantiate gps plugin. -->
+    <xacro:gps_plugin_macro
+      namespace="${namespace}"
+      gps_noise="true"
+      />
   </xacro:if>
 </robot>

Commit message: Update clover4.xacro

File: clover_description/urdf/clover/clover4.xacro (robot description, xacro)
@@ -16,5 +16,6 @@
   <xacro:if value="$(arg d435)">
     <xacro:sensor_d435 name="camera" topics_ns="camera" parent="base_link" publish_pointcloud="true">
-      <origin xyz="0 0 0.2" rpy="0 0 0" />
+      <!-- <origin xyz="0.0 0 0.2" rpy="0 0 0" />-->
+      <origin xyz="0.17 0 0" rpy="0 0 0" />
     </xacro:sensor_d435>
   </xacro:if>
